Commit message: update urdf

File: src/mrobot_description/urdf/mrobot.urdf (robot description, URDF)
Before this commit: robot mrobot, 6 links, 5 joints
Links:
- removed link front_castor_link
- added link base_footprint; visual box size=0.001 0.001 0.001
- added link front_caster_link, mass 0.001; collision sphere radius=0.0165; visual sphere radius=0.0165
- added link plate_1_link, mass 0.1; collision cylinder length=0.005 radius=0.13; visual cylinder length=0.005 radius=0.13
- added link plate_2_link, mass 0.01; collision cylinder length=0.005 radius=0.13; visual cylinder length=0.005 radius=0.13
- added link standoff_2in_1_link, mass 0.001; collision box size=0.01 0.01 0.07; visual box size=0.01 0.01 0.07
- added link standoff_2in_2_link, mass 0.001; collision box size=0.01 0.01 0.07; visual box size=0.01 0.01 0.07
- added link standoff_2in_3_link, mass 0.001; collision box size=0.01 0.01 0.07; visual box size=0.01 0.01 0.07
- added link standoff_2in_4_link, mass 0.001; collision box size=0.01 0.01 0.07; visual box size=0.01 0.01 0.07
- added link standoff_2in_5_link, mass 0.001; collision box size=0.01 0.01 0.07; visual box size=0.01 0.01 0.07
- added link standoff_2in_6_link, mass 0.001; collision box size=0.01 0.01 0.07; visual box size=0.01 0.01 0.07
- added link standoff_2in_7_link, mass 0.001; collision box size=0.01 0.01 0.07; visual box size=0.01 0.01 0.07
- added link standoff_2in_8_link, mass 0.001; collision box size=0.01 0.01 0.07; visual box size=0.01 0.01 0.07
- link base_link: mass None -> 2; geometry collision cylinder length=0.005 radius=0.13; visual cylinder length=0.005 radius=0.13
- link left_motor: mass None -> 0.1; geometry collision cylinder length=0.08 radius=0.02; visual cylinder length=0.08 radius=0.02
- link left_wheel_link: mass None -> 0.01; geometry collision cylinder length=0.017 radius=0.033; visual cylinder length=0.017 radius=0.033
- link right_motor: mass None -> 0.1; geometry collision cylinder length=0.08 radius=0.02; visual cylinder length=0.08 radius=0.02
- link right_wheel_link: mass None -> 0.01; geometry collision cylinder length=0.017 radius=0.033; visual cylinder length=0.017 radius=0.033
Joints:
- removed joint front_castor_joint
- added joint base_footprint_joint: type fixed, parent base_footprint, child base_link, origin xyz=0 0 0.033 rpy=0 0 0
- added joint front_caster_joint: type fixed, parent base_link, child front_caster_link, origin xyz=0.1135 0 -0.0165 rpy=0 0 0
- added joint plate_1_joint: type fixed, parent base_link, child plate_1_link, origin xyz=0 0 0.07 rpy=0 0 0
- added joint plate_2_joint: type fixed, parent plate_1_link, child plate_2_link, origin xyz=0 0 0.07 rpy=0 0 0
- added joint standoff_2in_1_joint: type fixed, parent base_link, child standoff_2in_1_link, origin xyz=-0.09 -0.07 0.035 rpy=0 0 0
- added joint standoff_2in_2_joint: type fixed, parent base_link, child standoff_2in_2_link, origin xyz=-0.09 0.07 0.035 rpy=0 0 0
- added joint standoff_2in_3_joint: type fixed, parent base_link, child standoff_2in_3_link, origin xyz=0.06 -0.1 0.035 rpy=0 0 0
- added joint standoff_2in_4_joint: type fixed, parent base_link, child standoff_2in_4_link, origin xyz=0.06 0.1 0.035 rpy=0 0 0
- added joint standoff_2in_5_joint: type fixed, parent standoff_2in_1_link, child standoff_2in_5_link, origin xyz=0 0 0.07 rpy=0 0 0
- added joint standoff_2in_6_joint: type fixed, parent standoff_2in_2_link, child standoff_2in_6_link, origin xyz=0 0 0.07 rpy=0 0 0
- added joint standoff_2in_7_joint: type fixed, parent standoff_2in_3_link, child standoff_2in_7_link, origin xyz=0 0 0.07 rpy=0 0 0
- added joint standoff_2in_8_joint: type fixed, parent standoff_2in_4_link, child standoff_2in_8_link, origin xyz=0 0 0.07 rpy=0 0 0
